File: hw/kicad/nop.kicad_sch (KiCad schematic)
At the start: 45 parts, among them J1 SD Card, J2 PS/2, U1 W65C02S, U10 TMS9118A, U11 62256, U12 74HCT04, U13 74HCT574, U14 74HCT574, U15 74HCT574, U16 74HCT14, U17 74HC595, U18 74HC595, U2 ATF16V8, U3 62256, U4 62256, U5 74HCT00, U6 2864, U7 74HCT273, U8 74HCT00, U9 W65C22S

Commit message: vm: proper ps2
Parts:
- U17, U18: value 74HC595 -> 74HCT595
Other:
- moved on the sheet: J1, R1
Changed lines of the file:
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@@
 	)
 	(no_connect
-		(at 214.63 234.95)
+		(at 213.36 234.95)
 	)
 	(no_connect
@@
 	(wire
 		(pts
-			(xy 180.34 237.49) (xy 182.88 237.49)
+			(xy 180.34 237.49) (xy 181.61 237.49)
 		)
 		(stroke
@@
 	(wire
 		(pts
+			(xy 213.36 340.36) (xy 214.63 340.36)
+		)
+		(stroke
+			(width 0)
+			(type default)
+		)
+	)
+	(wire
+		(pts
 			(xy 477.52 88.9) (xy 473.71 88.9)
 		)
@@
 	(wire
 		(pts
-			(xy 180.34 257.81) (xy 182.88 257.81)
+			(xy 180.34 257.81) (xy 181.61 257.81)
 		)
 		(stroke
@@
 	(wire
 		(pts
+			(xy 213.36 347.98) (xy 214.63 347.98)
+		)
+		(stroke
+			(width 0)
+			(type default)
+		)
+	)
+	(wire
+		(pts
 			(xy 167.64 154.94) (xy 167.64 151.13)
 		)
@@
 	(wire
 		(pts
-			(xy 213.36 234.95) (xy 214.63 234.95)
+			(xy 212.09 234.95) (xy 213.36 234.95)
 		)
 		(stroke
@@
 	(wire
 		(pts
-			(xy 180.34 255.27) (xy 182.88 255.27)
+			(xy 180.34 255.27) (xy 181.61 255.27)
 		)
 		(stroke
@@
 		)
 	)
+	(wire
+		(pts
+			(xy 213.36 337.82) (xy 214.63 337.82)
+		)
+		(stroke
+			(width 0)
+			(type default)
+		)
+	)
 	(bus
 		(pts
@@
 	(wire
 		(pts
+			(xy 213.36 355.6) (xy 214.63 355.6)
+		)
+		(stroke
+			(width 0)
+			(type default)
+		)
+	)
+	(wire
+		(pts
 			(xy 420.37 55.88) (xy 420.37 45.72)
 		)
@@
 		)
 	)
+	(wire
+		(pts
+			(xy 213.36 345.44) (xy 214.63 345.44)
+		)
+		(stroke
+			(width 0)
+			(type default)
+		)
+	)
 	(bus
 		(pts
@@
 	(wire
 		(pts
-			(xy 177.8 234.95) (xy 182.88 234.95)
+			(xy 177.8 234.95) (xy 181.61 234.95)
 		)
 		(stroke
@@
 	(wire
 		(pts
-			(xy 182.88 250.19) (xy 177.8 250.19)
+			(xy 181.61 250.19) (xy 177.8 250.19)
 		)
 		(stroke
@@
 	(wire
 		(pts
-			(xy 213.36 237.49) (xy 218.44 237.49)
+			(xy 212.09 237.49) (xy 217.17 237.49)
 		)
 		(stroke
@@
 	(wire
 		(pts
-			(xy 180.34 240.03) (xy 182.88 240.03)
+			(xy 180.34 240.03) (xy 181.61 240.03)
 		)
 		(stroke
@@
 		)
 	)
+	(wire
+		(pts
+			(xy 213.36 350.52) (xy 214.63 350.52)
+		)
+		(stroke
+			(width 0)
+			(type default)
+		)
+	)
 	(bus
 		(pts
@@
 	(wire
 		(pts
-			(xy 176.53 242.57) (xy 182.88 242.57)
+			(xy 176.53 242.57) (xy 181.61 242.57)
 		)
 		(stroke
@@
 	(wire
 		(pts
-			(xy 175.26 247.65) (xy 182.88 247.65)
+			(xy 175.26 247.65) (xy 181.61 247.65)
 		)
 		(stroke
@@
 	(wire
 		(pts
+			(xy 213.36 342.9) (xy 214.63 342.9)
+		)
+		(stroke
+			(width 0)
+			(type default)
+		)
+	)
+	(wire
+		(pts
 			(xy 182.88 52.07) (xy 177.8 52.07)
 		)
@@
 			)
 		)
-		(property "Value" "74HC595"
+		(property "Value" "74HCT595"
 			(at 162.1633 327.66 0)
 			(effects
@@
 	(symbol
 		(lib_id "Device:R_US")
-		(at 218.44 241.3 180)
+		(at 217.17 241.3 180)
 		(unit 1)
 		(exclude_from_sim no)
@@
 		(fields_autoplaced yes)
 		(property "Reference" "R1"
-			(at 220.98 240.0299 0)
+			(at 219.71 240.0299 0)
 			(effects
 				(font
@@
 		)
 		(property "Value" "10K"
-			(at 220.98 242.5699 0)
+			(at 219.71 242.5699 0)
 			(effects
 				(font
@@
 		)
 		(property "Footprint" "Resistor_THT:R_Axial_DIN0204_L3.6mm_D1.6mm_P7.62mm_Horizontal"
-			(at 217.424 241.046 90)
+			(at 216.154 241.046 90)
 			(effects
 				(font
@@
 		)
 		(property "Datasheet" "~"
-			(at 218.44 241.3 0)
+			(at 217.17 241.3 0)
 			(effects
 				(font
@@
 		)
 		(property "Description" "Resistor, US symbol"
-			(at 218.44 241.3 0)
+			(at 217.17 241.3 0)
 			(effects
 				(font
@@
 	(symbol
 		(lib_id "power:GND")
-		(at 218.44 245.11 0)
+		(at 217.17 245.11 0)
 		(unit 1)
 		(exclude_from_sim no)
@@
 		(fields_autoplaced yes)
 		(property "Reference" "#PWR024"
-			(at 218.44 251.46 0)
+			(at 217.17 251.46 0)
 			(effects
 				(font
@@
 		)
 		(property "Value" "GND"
-			(at 218.44 250.19 0)
+			(at 217.17 250.19 0)
 			(effects
 				(font
@@
 		)
 		(property "Footprint" ""
-			(at 218.44 245.11 0)
+			(at 217.17 245.11 0)
 			(effects
 				(font
@@
 		)
 		(property "Datasheet" ""
-			(at 218.44 245.11 0)
+			(at 217.17 245.11 0)
 			(effects
 				(font
@@
 		)
 		(property "Description" "Power symbol creates a global label with name \"GND\" , ground"
-			(at 218.44 245.11 0)
+			(at 217.17 245.11 0)
 			(effects
 				(font
@@
 			)
 		)
-		(property "Value" "74HC595"
+		(property "Value" "74HCT595"
 			(at 205.3433 327.66 0)
 			(effects
@@
 	(symbol
 		(lib_id "power:+5V")
-		(at 198.12 224.79 0)
+		(at 196.85 224.79 0)
 		(unit 1)
 		(exclude_from_sim no)
@@
 		(fields_autoplaced yes)
 		(property "Reference" "#PWR023"
-			(at 198.12 228.6 0)
+			(at 196.85 228.6 0)
 			(effects
 				(font
@@
 		)
 		(property "Value" "+5V"
-			(at 198.12 219.71 0)
+			(at 196.85 219.71 0)
 			(effects
 				(font
@@
 		)
 		(property "Footprint" ""
-			(at 198.12 224.79 0)
+			(at 196.85 224.79 0)
 			(effects
 				(font
@@
 		)
 		(property "Datasheet" ""
-			(at 198.12 224.79 0)
+			(at 196.85 224.79 0)
 			(effects
 				(font
@@
 		)
 		(property "Description" "Power symbol creates a global label with name \"+5V\""
-			(at 198.12 224.79 0)
+			(at 196.85 224.79 0)
 			(effects
 				(font
@@
 	(symbol
 		(lib_id "power:GND")
-		(at 198.12 265.43 0)
+		(at 196.85 265.43 0)
 		(unit 1)
 		(exclude_from_sim no)
@@
 		(fields_autoplaced yes)
 		(property "Reference" "#PWR022"
-			(at 198.12 271.78 0)
+			(at 196.85 271.78 0)
 			(effects
 				(font
@@
 		)
 		(property "Value" "GND"
-			(at 198.12 270.51 0)
+			(at 196.85 270.51 0)
 			(effects
 				(font
@@
 		)
 		(property "Footprint" ""
-			(at 198.12 265.43 0)
+			(at 196.85 265.43 0)
 			(effects
 				(font
@@
 		)
 		(property "Datasheet" ""
-			(at 198.12 265.43 0)
+			(at 196.85 265.43 0)
 			(effects
 				(font
@@
 		)
 		(property "Description" "Power symbol creates a global label with name \"GND\" , ground"
-			(at 198.12 265.43 0)
+			(at 196.85 265.43 0)
 			(effects
 				(font
@@
 	(symbol
 		(lib_id "Connector:SD_Card_Receptacle")
-		(at 198.12 245.11 0)
+		(at 196.85 245.11 0)
 		(unit 1)
 		(exclude_from_sim no)
@@
 		(dnp no)
 		(property "Reference" "J1"
-			(at 200.2633 222.25 0)
+			(at 198.9933 222.25 0)
 			(effects
 				(font
@@
 		)
 		(property "Value" "SD Card"
-			(at 200.2633 224.79 0)
+			(at 198.9933 224.79 0)
 			(effects
 				(font
@@
 		)
 		(property "Footprint" "Connector_Card:SD_Hirose_DM1AA_SF_PEJ82"
-			(at 207.01 248.412 0)
+			(at 205.74 248.412 0)
 			(effects
 				(font
@@
 		)
 		(property "Datasheet" "http://portal.fciconnect.com/Comergent//fci/drawing/10067847.pdf"
-			(at 198.12 245.11 0)
+			(at 196.85 245.11 0)
 			(effects
 				(font
@@
 		)
 		(property "Description" "SD card receptacle"
-			(at 198.12 245.11 0)
+			(at 196.85 245.11 0)
 			(effects
 				(font

Commit message: layout attempt 1
Parts:
- added C19, C20, C21, C22, C23, C28, C37, C38: 0.1uF, Capacitor_THT:C_Disc_D7.5mm_W4.4mm_P5.00mm, symbol Device:C
- added C26, C27: 27pF, Capacitor_THT:C_Disc_D7.5mm_W4.4mm_P5.00mm, symbol Device:C
- added C29: 30pF, Capacitor_THT:C_Disc_D7.5mm_W4.4mm_P5.00mm, symbol Device:C
- added C30: 10pF, Capacitor_THT:C_Disc_D7.5mm_W4.4mm_P5.00mm, symbol Device:C
- added C31, C32, C33, C34, C36: 10uF, Capacitor_THT:CP_Radial_D5.0mm_P2.50mm, symbol Device:C_Polarized
- added C35: 220uF, Capacitor_THT:CP_Radial_D5.0mm_P2.50mm, symbol Device:C_Polarized
- added FB1: FerriteBead, Inductor_THT:L_Axial_L5.3mm_D2.2mm_P7.62mm_Horizontal_Vishay_IM-1, symbol Device:FerriteBead
- added J3: TV, Connector_PinHeader_2.54mm:PinHeader_1x02_P2.54mm_Vertical, symbol Connector:Conn_Coaxial
- added J4: RS232, Connector_PinHeader_2.54mm:PinHeader_2x05_P2.54mm_Vertical, symbol Connector:DE9_Pins
- added J5: POWER, Connector_PinHeader_2.54mm:PinHeader_1x02_P2.54mm_Vertical, symbol Connector:Conn_01x02_Pin
- added LS1: Speaker, Connector_PinHeader_2.54mm:PinHeader_1x02_P2.54mm_Vertical, symbol Device:Speaker
- added Q1: 2N4401, Package_TO_SOT_THT:TO-92, symbol Transistor_BJT:Q_NPN_EBC
- added R10, R11, R12, R13, R14, R15, R16, R17, R7, R8: 10K, Resistor_THT:R_Axial_DIN0204_L3.6mm_D1.6mm_P7.62mm_Horizontal, symbol Device:R_US
- added R18: 10R, Resistor_THT:R_Axial_DIN0204_L3.6mm_D1.6mm_P7.62mm_Horizontal, symbol Device:R_US
- added R5: 75K, Resistor_THT:R_Axial_DIN0204_L3.6mm_D1.6mm_P7.62mm_Horizontal, symbol Device:R_US
- added R6: 470K, Resistor_THT:R_Axial_DIN0204_L3.6mm_D1.6mm_P7.62mm_Horizontal, symbol Device:R_US
- added R9: 1M, Resistor_THT:R_Axial_DIN0204_L3.6mm_D1.6mm_P7.62mm_Horizontal, symbol Device:R_US
- added RV1: VOL, Connector_PinHeader_2.54mm:PinHeader_1x03_P2.54mm_Vertical, symbol Device:R_Potentiometer_US
- added U19: 16550, Package_DIP:DIP-40_W15.24mm_Socket, symbol Interface_UART:16550
- added U20: MAX232, Package_DIP:DIP-16_W7.62mm_Socket, symbol Interface_UART:MAX232
- added U21: 74HCT00, Package_DIP:DIP-14_W7.62mm_Socket, symbol 74xx:74HCT00
- added U22: SN76489AN, Package_DIP:DIP-16_W7.62mm_Socket, symbol Audio:SN76489AN
- added U23: LM386, Package_DIP:DIP-8_W7.62mm_Socket, symbol Amplifier_Audio:LM386
- added Y1: 10.738635Mhz, Crystal:Crystal_HC49-4H_Vertical, symbol Device:Crystal
- added Y2: 11.0592Mhz, Crystal:Crystal_HC49-4H_Vertical, symbol Device:Crystal
- added Y4: 1Mhz, Oscillator:Oscillator_DIP-14, symbol Oscillator:DGOF5S3
- J1: footprint Connector_Card:SD_Hirose_DM1AA_SF_PEJ82 -> Connector_Card:SD_Kyocera_145638009511859+
- renumbered C20 to C24, C19 to C25
Connections:
- net +5V: now also C19.1, C20.1, C21.1, C22.1, C23.1, C33.2, FB1.1, J5.1 (Pin_1), R11.2, R12.2, R14.2, R15.2, R16.2, R17.2, R7.2, U19.40 (VCC), U20.16 (VCC), U21.14 (VCC), U22.16 (V_{CC}), U23.6 (V+), Y4.14 (Vcc); no longer U9.24 (CS1)
- net GND: now also J1.12 (SHELL1), J1.13 (SHELL2), U14.1 (OE), U15.1 (OE), C19.2, C20.2, C21.2, C22.2, C23.2, C26.2, C27.2, C28.2, C29.2, C30.2, C34.1, C38.2, J3.2 (Ext), J4.5, J5.2 (Pin_2), LS1.2, R13.1, R18.1, R5.1, R6.1, R8.1, RV1.3, U19.20 (GND), U20.15 (GND), U21.7 (GND), U22.8 (GND), U23.2 (-), U23.4 (GND), Y4.7 (GND)
- net a0: now also U19.28 (A0)
- net a1: now also U19.27 (A1)
- net a2: now also U19.26 (A2)
- net d0: now also U19.1 (D0), U22.3 (D0)
- net d1: now also U19.2 (D1), U22.2 (D1)
- net d2: now also U19.3 (D2), U22.1 (D2)
- net d3: now also U19.4 (D3), U22.15 (D3)
- net d4: now also U19.5 (D4), U22.13 (D4)
- net d5: now also U19.6 (D5), U22.12 (D5)
- net d6: now also U19.7 (D6), U22.11 (D6)
- net d7: now also U19.8 (D7), U22.10 (D7)
- net r/~{w}: now also U8.12, U21.2, U22.5 (~{WE})
- net va0: now also U11.10 (A0), U14.18 (Q1); no longer U10.10 (AD0)
- net va1: now also U11.9 (A1), U14.17 (Q2); no longer U10.9 (AD1)
- net va2: now also U11.8 (A2), U14.16 (Q3); no longer U10.8 (AD2)
- net va3: now also U11.7 (A3), U14.15 (Q4); no longer U10.7 (AD3)
- net va4: now also U11.6 (A4), U14.14 (Q5); no longer U10.6 (AD4)
- net va5: now also U11.5 (A5), U14.13 (Q6); no longer U10.5 (AD5)
- net va6: now also U11.4 (A6), U14.12 (Q7); no longer U10.4 (AD6)
- net va7: now also U11.3 (A7), U15.18 (Q1); no longer U10.3 (AD7)
- net vd0: now also U13.19 (Q0)
- net vd1: now also U13.18 (Q1)
- net vd2: now also U13.17 (Q2)
- net vd3: now also U13.16 (Q3)
- net vd4: now also U13.15 (Q4)
- net vd5: now also U13.14 (Q5)
- net vd6: now also U13.13 (Q6)
- net vd7: now also U13.12 (Q7)
- net ~{dev2}: now also U19.14 (~{CS2}), U22.6 (~{CE})
- net ~{irq}: now also U21.11; no longer U9.21 (~{IRQ})
- net ~{res}: now also U12.13
- net va13: now reaches U11.1 (A14)
- net va13: now also U11.26 (A13), U15.12 (Q7)
- net va12: now reaches U11.2 (A12)
- net va12: now also U15.13 (Q6)
- net at U11.20 (~{CS}): now also U10.2 (~{CAS}), U12.3
- net va10: now reaches U11.21 (A10)
- net va10: now also U15.15 (Q4)
- net at U11.22 (~{OE}): now also U12.10, U13.11 (Cp)
- net va11: now reaches U11.23 (A11)
- net va11: now also U15.14 (Q5)
- net va9: now reaches U11.24 (A9)
- net va9: now also U15.16 (Q3)
- net va8: now reaches U11.25 (A8)
- net va8: now also U15.17 (Q2)
- net at U11.27 (~{WE}): now also U10.11 (R/~{W}), U12.11, U13.1 (OE)
- net at U10.36 (COMVID): now also Q1.2 (B), R6.2
- net aclk: now reaches U10.38 (CPUCLK)
- net aclk: now also U22.14 (CLOCK)
- net at U10.39 (XTAL2): now also C26.1, Y1.2
- net at U10.40 (XTAL1): now also C27.1, Y1.1
- net at U14.11 (Cp): now also U12.2
- net ad0: now reaches U14.2 (D0)
- net ad0: now also U10.10 (AD0), U13.2 (D0), U15.2 (D0)
- net ad1: now reaches U14.3 (D1)
- net ad1: now also U10.9 (AD1), U13.3 (D1), U15.3 (D1)
- net ad2: now reaches U14.4 (D2)
- net ad2: now also U10.8 (AD2), U13.4 (D2), U15.4 (D2)
- net ad3: now reaches U14.5 (D3)
- net ad3: now also U10.7 (AD3), U13.5 (D3), U15.5 (D3)
- net ad4: now reaches U14.6 (D4)
- net ad4: now also U10.6 (AD4), U13.6 (D4), U15.6 (D4)
- net ad5: now reaches U14.7 (D5)
- net ad5: now also U10.5 (AD5), U13.7 (D5), U15.7 (D5)
- net ad6: now reaches U14.8 (D6)
- net ad6: now also U10.4 (AD6), U13.8 (D6), U15.8 (D6)
- net ad7: now reaches U14.9 (D7)
- net ad7: now also U10.3 (AD7), U13.9 (D7), U15.9 (D7)
- net at U1.2 (RDY): now also R14.1
- net at U1.36 (BE): now also R15.1
- net clk: now reaches U1.37 (ϕ0)
- net clk: now also U8.13, U21.1, Y4.8 (OUT)
- net at U1.38 (~{SO}): now also R16.1
- net at U8.11: now also U19.21 (~{RD})
- net at U15.11 (Cp): now also U12.8
- net at U12.12: now also U19.35 (MR)
- net at U12.4: now also U12.5
- net at J1.11 (WRITE_PROTECT), R1.2: now also J1.10 (CARD_DETECT)
- net vr/~{w}: no longer names the net of U12.1
- net vr/~{w}: now also U10.1 (~{RAS}); no longer U10.11 (R/~{W})
- removed net v~{r}/w: U12.13, U12.2
- removed net ~{cas}: U10.1 (~{RAS}), U10.2 (~{CAS})
- new net: J4.2, U20.14 (T1OUT)
- new net: J4.3, U20.13 (R1IN)
- new net: J4.7, U20.7 (T2OUT)
- new net: J4.8, U20.8 (R2IN)
- new net: R11.1, U9.24 (CS1)
- new net: U21.12, U21.6
- new net: C28.1, FB1.2, Q1.3 (C)
- new net: C30.1, R9.2, U19.16 (XIN), Y2.1
- new net: C29.1, R10.2, R9.1, Y2.2
- new net: J3.1 (In), Q1.1 (E), R5.2
- new net: U19.18 (~{WR}), U21.3
- new net: U19.10 (SIN), U20.11 (T1IN)
- new net: U19.11 (SOUT), U20.12 (R1OUT)
- new net: R7.1, U19.12 (CS0), U19.13 (CS1)
- new net: U19.15 (~{BAUDOUT}), U19.9 (RCLK)
- new net: R10.1, U19.17 (XOUT)
- new net: R8.2, U19.19 (WR), U19.22 (RD), U19.25 (~{ADS})
- new net: U19.32 (~{RTS}), U20.10 (T2IN)
- new net: U19.36 (~{CTS}), U20.9 (R2OUT)
- new net: R13.2, U19.37 (~{DSR}), U19.38 (~{DCD}), U19.39 (~{RI})
- new net: C31.1, U20.1 (C1+)
- new net: C33.1, U20.2 (VS+)
- new net: C31.2, U20.3 (C1-)
- new net: C32.1, U20.4 (C2+)
- new net: C32.2, U20.5 (C2-)
- new net: C34.2, U20.6 (VS-)
- new net: U21.13, U21.8
- new net: C36.1, U23.1 (GAIN)
- new net: C36.2, U23.8 (GAIN)
- new net: C35.1, C37.1, U23.5
- new net: C35.2, LS1.1
- new net: C38.1, U23.7 (BYPASS)
- new net: R12.1, U21.10
- new net: C37.2, R18.2
- new net: RV1.2, U23.3 (+)
- new net: R17.1, U22.4 (READY)
- new net: RV1.1, U22.7 (AUDIO_OUT)
- new net i1: U19.30 (INTR), U21.9
- new net ~{i0}: U21.4, U21.5, U9.21 (~{IRQ})
- no-connect marks 24 -> 38
Other:
- moved on the sheet: C1, C10, C11, C12, C13, C14, C15, C16, C5, C8, R1, U1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

Commit message: try routing again
Parts:
- removed C37: 0.1uF, Capacitor_THT:C_Disc_D7.5mm_W4.4mm_P5.00mm, symbol Device:C
- removed J1: SD Card, Connector_Card:SD_Kyocera_145638009511859+, symbol Connector:SD_Card_Receptacle
- removed R1: 10K, Resistor_THT:R_Axial_DIN0204_L3.6mm_D1.6mm_P7.62mm_Horizontal, symbol Device:R_US
- added C12, C27, C28: 0.1uF, Capacitor_THT:C_Disc_D7.5mm_W4.4mm_P5.00mm, symbol Device:C
- added J3: SD Breakout, Connector_PinHeader_2.54mm:PinHeader_1x08_P2.54mm_Vertical, symbol Connector:Conn_01x08_Pin
- added J4: Reset, Connector_PinHeader_2.54mm:PinHeader_1x02_P2.54mm_Vertical, symbol Connector:Conn_01x02_Pin
- added U12: (no value), Package_TO_SOT_THT:TO-92, symbol nop:DS1813
- added Y2: 4Mhz, Oscillator:Oscillator_DIP-8, symbol Oscillator:CXO_DIP8
- RV1: value VOL -> 10K
- renumbered C2 to C10, C7 to C11, C5 to C13, C21 to C14, C8 to C15, C13 to C16, C14 to C17, C15 to C18, C12 to C19, C10 to C2, C38 to C20, C18 to C21, C17 to C22, C16 to C23, C20 to C24, C24 to C26, C36 to C29, C9 to C3, C23 to C30, C35 to C31, C30 to C32, C29 to C33, C28 to C34, C27 to C35, C31 to C36, C26 to C37, C32 to C38, C33 to C39, C19 to C4, C34 to C40, C22 to C5, C3 to C6, C4 to C7, C6 to C8, C11 to C9, J2 to J1, J5 to J2, J3 to J5, J4 to J6, R2 to R1, R18 to R10, R9 to R11, R7 to R12, R8 to R13, R10 to R14, R5 to R15, R6 to R16, R13 to R17, R3 to R2, R4 to R3, R11 to R4, R15 to R5, R16 to R6, R14 to R7, R12 to R8, R17 to R9, U2 to U10, U7 to U11, U21 to U13, U5 to U13, U8 to U13, U21 to U14, U5 to U14, U8 to U15, U21 to U15, U13 to U16, U14 to U17, U15 to U18, U12 to U19, U10 to U2, U23 to U20, U18 to U21, U17 to U22, U16 to U23, U20 to U24, U9 to U3, U19 to U4, U22 to U5, U3 to U6, U4 to U7, U6 to U8, U11 to U9, Y4 to Y1, Y2 to Y3, Y1 to Y4
Connections:
- net +5V: now also C12.1, C27.1, C28.1, J3.8 (5v), U12.2 (VCC), Y2.8 (Vcc); no longer C30.1
- net GND: now also C12.2, C27.2, C28.2, J3.6 (GND), J4.2 (Pin_2), U12.3 (GND), Y2.4 (GND); no longer C30.2
- net ~{dev1}: now also U4.14 (~{CS2})
- net ~{dev2}: no longer U4.14 (~{CS2})
- net ~{res}: now also J4.1 (Pin_1), U12.1 (~{RST})
- net at U3.2 (PA0): now also J3.2 (CS)
- net at U3.3 (PA1): now also J3.5 (CLK)
- net at U3.4 (PA2): now also J3.3 (DI); no longer U3.9 (PA7)
- net at U4.10 (SIN): now also U24.12 (R1OUT); no longer U24.11 (T1IN)
- net at U4.11 (SOUT): now also U24.11 (T1IN); no longer U24.12 (R1OUT)
- net at C31.1, U20.5: now also C30.1
- net at R10.2: now also C30.2
- net aclk: no longer names the net of U2.38 (CPUCLK)
- net aclk: no longer U5.14 (CLOCK)
- new net: J3.4 (DO), U3.9 (PA7)
- new net: U5.14 (CLOCK), Y2.5 (OUT)
- no-connect marks 38 -> 40
Other:
- moved on the sheet: C1, C10, C11, C13, C14, C15, C16, C17, C18, C19, C2, C20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

Commit message: vm/hw: simplify hw. remove bank switch flip-flop in favor of VIA pin
Parts:
- removed C11, C14, C28: 0.1uF, Capacitor_THT:C_Disc_D7.5mm_W4.4mm_P5.00mm, symbol Device:C
- removed R8: 10K, Resistor_THT:R_Axial_DIN0204_L3.6mm_D1.6mm_P7.62mm_Horizontal, symbol Device:R_US
- removed U11: 74HCT273, Package_DIP:DIP-20_W7.62mm_Socket, symbol 74xx:74HCT273
- removed U14: 74HCT00, Package_DIP:DIP-14_W7.62mm_Socket, symbol 74xx:74HCT00
- removed Y2: 4Mhz, Oscillator:Oscillator_DIP-8, symbol Oscillator:CXO_DIP8
- added R18: 10K, Resistor_THT:R_Axial_DIN0204_L3.6mm_D1.6mm_P7.62mm_Horizontal, symbol Device:R_US
Connections:
- net bk0 is gone; now on net a13: U7.26 (A13)
- net bk1 is gone; now on net bk: U7.1 (A14)
- net ram is gone; now on net ~{ramlo}: U10.13 (I/O)
- net +5V: now also U13.5
- net GND: now also R18.1
- net clk: now also U15.2, U15.4; no longer U15.1, U15.13
- net dev0: now also U10.15 (I/O), U13.12, U15.13; no longer U10.14 (I/O), U15.5, U15.9
- net i1: now also U13.4; no longer U13.9
- net r/~{w}: now also U15.1, U15.5, U19.13; no longer U13.12, U13.13, U15.2, U15.4
- net ~{dev1}: now also U10.16 (I/O); no longer U10.15 (I/O)
- net ~{dev2}: now also U10.17 (I/O); no longer U10.16 (I/O)
- net ~{dev3}: now also U10.18 (I/O); no longer U10.17 (I/O)
- net ~{dev4}: now also U10.19 (I/O); no longer U10.18 (I/O)
- net ~{i0}: now also U13.1, U13.2; no longer U13.4, U13.5
- net ~{irq}: now also U13.8
- net ~{res}: now also U15.10, U15.9; no longer U19.13
- net at U2.14 (~{CSW}): now also U13.11; no longer U15.8
- net at U2.15 (~{CSR}): now also U15.11; no longer U15.6
- net aclk: now reaches U2.38 (CPUCLK)
- net aclk: now also U5.14 (CLOCK)
- net bk: now reaches U3.39 (CA2)
- net bk: now also R18.2
- net ~{ramlo}: now reaches U6.20 (~{CS}), U6.22 (~{OE})
- net at U13.6: now also U13.10
- net at U4.21 (~{RD}): now also U15.3; no longer U15.11
- net at U4.35 (MR): now also U15.8; no longer U19.12
- net ~{ramhi}: now reaches U7.20 (~{CS}), U7.22 (~{OE})
- net ~{ramhi}: now also U10.14 (I/O)
- net at U4.18 (~{WR}): now also U15.6; no longer U15.3
- net at U13.3: now also U13.9
- removed net dev5: U10.19 (I/O), U13.2
- removed net ~{r}/w: U13.1, U13.11, U15.10
- new net: U13.13, U19.12
- no-connect marks 40 -> 37
Other:
- moved on the sheet: U13A

Commit message: hw: update pcb
Parts:
- J2: value POWER -> +5V
Connections:
- net ~{dev1}: no longer U4.14 (~{CS2})
- net ~{dev3}: now also U4.14 (~{CS2})
Changed lines of the file:
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@@
 	(wire
 		(pts
-			(xy 459.74 297.18) (xy 473.71 297.18)
+			(xy 461.01 297.18) (xy 473.71 297.18)
 		)
 		(stroke
@@
 	(wire
 		(pts
-			(xy 459.74 287.02) (xy 459.74 297.18)
+			(xy 461.01 287.02) (xy 461.01 297.18)
 		)
 		(stroke
@@
 	(wire
 		(pts
+			(xy 461.01 287.02) (xy 459.74 287.02)
+		)
+		(stroke
+			(width 0)
+			(type default)
+		)
+	)
+	(wire
+		(pts
 			(xy 698.5 314.96) (xy 584.2 314.96)
 		)
@@
 		)
 	)
-	(global_label "~{dev1}"
+	(global_label "~{dev3}"
 		(shape input)
 		(at 421.64 71.12 180)
@@
 			)
 		)
-		(property "Value" "POWER"
+		(property "Value" "+5V"
 			(at 22.225 175.26 0)
 			(show_name no)

Commit message: hw: complete layout
Parts:
- removed J2: +5V, Connector_PinHeader_2.54mm:PinHeader_1x02_P2.54mm_Vertical, symbol Connector:Conn_01x02_Pin
- added C11: 0.1uF, Capacitor_THT:C_Disc_D7.5mm_W4.4mm_P5.00mm, symbol Device:C
- added J2: LM73100 Breakout, Connector_PinHeader_2.54mm:PinHeader_1x09_P2.54mm_Vertical, symbol Connector:Conn_01x09_Pin
- added J7: Ext, Connector_PinHeader_2.54mm:PinHeader_2x10_P2.54mm_Vertical, symbol Connector_Generic:Conn_02x10_Counter_Clockwise
- added J8: Vin, Connector_PinHeader_2.54mm:PinHeader_1x01_P2.54mm_Vertical, symbol Connector:Conn_01x01_Pin
- added R19: 91K, Resistor_THT:R_Axial_DIN0204_L3.6mm_D1.6mm_P7.62mm_Horizontal, symbol Device:R_US
- added R20: 27K, Resistor_THT:R_Axial_DIN0204_L3.6mm_D1.6mm_P7.62mm_Horizontal, symbol Device:R_US
- added R8: 10K, Resistor_THT:R_Axial_DIN0204_L3.6mm_D1.6mm_P7.62mm_Horizontal, symbol Device:R_US
- U12: value (none) -> DS1813
Connections:
- net +5V: now also J2.9 (Vout), J7.20 (Pin_20), R8.2; no longer U13.5
- net GND: now also C11.1, J2.2 (GND), J7.10 (Pin_10), R20.2
- net a0: now also J7.18 (Pin_18)
- net a1: now also J7.17 (Pin_17)
- net a2: now also J7.16 (Pin_16)
- net a3: now also J7.15 (Pin_15)
- net d0: now also J7.1 (Pin_1)
- net d1: now also J7.2 (Pin_2)
- net d2: now also J7.3 (Pin_3)
- net d3: now also J7.4 (Pin_4)
- net d4: now also J7.5 (Pin_5)
- net d5: now also J7.6 (Pin_6)
- net d6: now also J7.7 (Pin_7)
- net d7: now also J7.8 (Pin_8)
- net i1: now also U13.5; no longer U13.4
- net r/~{w}: now also J7.13 (Pin_13)
- net ~{dev4}: now also J7.9 (Pin_9)
- net ~{res}: now also J7.14 (Pin_14)
- net at U13.6: now also U13.9; no longer U13.10
- net at U13.3: now also U13.4; no longer U13.9
- new net: C11.2, J2.4 (OVLO), R19.1, R20.1
- new net: J2.1 (Vin), J8.1 (+5V), R19.2
- new net ~{i2}: R8.1, U13.10
- no-connect marks 37 -> 45
Other:
- moved on the sheet: C13, C15, U13E, U15E
