File: hw/kicad/nop.kicad_pcb (KiCad board)
At the start: 2 copper layers, 195.6 x 149.9 mm, 92 parts, among them J1 SD Card, J2 PS/2, J3 TV, J4 RS232, J5 POWER, Q1 2N4401, U1 W65C02S, U10 TMS9118A, U11 62256, U12 74HCT04, U13 74HCT574, U14 74HCT574, U15 74HCT574, U16 74HCT14, U17 74HCT595, U18 74HCT595, U19 16550, U2 ATF16V8, U20 MAX232, U21 74HCT00, U22 SN76489AN, U23 LM386, U3 62256, U4 62256, U5 74HCT00, U6 2864, U7 74HCT273, U8 74HCT00, U9 W65C22S, Y1 10.738635Mhz, Y2 11.0592Mhz, Y4 1Mhz

Commit message: try routing again
Parts:
- removed R18: 10R, Resistor_THT:R_Axial_DIN0204_L3.6mm_D1.6mm_P7.62mm_Horizontal
- added C39: 10uF, Capacitor_THT:CP_Radial_D5.0mm_P2.50mm, F.Cu at (384.3, 429.3)
- added C40: 10uF, Capacitor_THT:CP_Radial_D5.0mm_P2.50mm, F.Cu at (384.3, 435.8)
- added J6: RS232, Connector_PinHeader_2.54mm:PinHeader_2x05_P2.54mm_Vertical, F.Cu at (443.5, 363.3)
- added U24: MAX232, Package_DIP:DIP-16_W7.62mm_Socket, F.Cu at (431.6, 351.3)
- added Y3: 11.0592Mhz, Crystal:Crystal_HC49-4H_Vertical, F.Cu at (412.8, 439.1)
- C26, C27: value 27pF -> 0.1uF
- C29: value 30pF -> 10uF; footprint Capacitor_THT:C_Disc_D7.5mm_W4.4mm_P5.00mm -> Capacitor_THT:CP_Radial_D5.0mm_P2.50mm
- C30: value 10pF -> 0.1uF
- C31: value 10uF -> 220uF
- C32: value 10uF -> 10pF; footprint Capacitor_THT:CP_Radial_D5.0mm_P2.50mm -> Capacitor_THT:C_Disc_D7.5mm_W4.4mm_P5.00mm
- C33: value 10uF -> 30pF; footprint Capacitor_THT:CP_Radial_D5.0mm_P2.50mm -> Capacitor_THT:C_Disc_D7.5mm_W4.4mm_P5.00mm
- C34: value 10uF -> 0.1uF; footprint Capacitor_THT:CP_Radial_D5.0mm_P2.50mm -> Capacitor_THT:C_Disc_D7.5mm_W4.4mm_P5.00mm
- C35: value 220uF -> 27pF; footprint Capacitor_THT:CP_Radial_D5.0mm_P2.50mm -> Capacitor_THT:C_Disc_D7.5mm_W4.4mm_P5.00mm
- C37: value 0.1uF -> 27pF
- C38: value 0.1uF -> 10uF; footprint Capacitor_THT:C_Disc_D7.5mm_W4.4mm_P5.00mm -> Capacitor_THT:CP_Radial_D5.0mm_P2.50mm
- J1: value SD Card -> PS/2; footprint Connector_Card:SD_Kyocera_145638009511859+ -> Connector_PinHeader_2.54mm:PinHeader_1x06_P2.54mm_Vertical
- J2: value PS/2 -> POWER; footprint Connector_PinHeader_2.54mm:PinHeader_1x06_P2.54mm_Vertical -> Connector_PinHeader_2.54mm:PinHeader_1x02_P2.54mm_Vertical
- J3: value TV -> SD Breakout; footprint Connector_PinHeader_2.54mm:PinHeader_1x02_P2.54mm_Vertical -> Connector_PinHeader_2.54mm:PinHeader_1x08_P2.54mm_Vertical
- J4: value RS232 -> Reset; footprint Connector_PinHeader_2.54mm:PinHeader_2x05_P2.54mm_Vertical -> Connector_PinHeader_2.54mm:PinHeader_1x02_P2.54mm_Vertical
- J5: value POWER -> TV
- R10: value 10K -> 10R
- R11: value 10K -> 1M
- R15: value 10K -> 75K
- R16: value 10K -> 470K
- R3: value 10K -> 5.6K
- R4: value 5.6K -> 10K
- R5: value 75K -> 10K
- R6: value 470K -> 10K
- R9: value 1M -> 10K
- RV1: value VOL -> 10K
- U10: value TMS9118A -> ATF16V8; footprint Package_DIP:DIP-40_W15.24mm_Socket -> Package_DIP:DIP-20_W7.62mm_Socket
- U11: value 62256 -> 74HCT273; footprint Package_DIP:DIP-28_W15.24mm_Socket -> Package_DIP:DIP-20_W7.62mm_Socket
- U12: value 74HCT04 -> ~; footprint Package_DIP:DIP-14_W7.62mm_Socket -> Package_TO_SOT_THT:TO-92
- U13, U14, U15: value 74HCT574 -> 74HCT00; footprint Package_DIP:DIP-20_W7.62mm_Socket -> Package_DIP:DIP-14_W7.62mm_Socket
- U16: value 74HCT14 -> 74HCT574; footprint Package_DIP:DIP-14_W7.62mm_Socket -> Package_DIP:DIP-20_W7.62mm_Socket
- U17, U18: value 74HCT595 -> 74HCT574; footprint Package_DIP:DIP-16_W7.62mm_Socket -> Package_DIP:DIP-20_W7.62mm_Socket
- U19: value 16550 -> 74HCT04; footprint Package_DIP:DIP-40_W15.24mm_Socket -> Package_DIP:DIP-14_W7.62mm_Socket
- U2: value ATF16V8 -> TMS9118A; footprint Package_DIP:DIP-20_W7.62mm_Socket -> Package_DIP:DIP-40_W15.24mm_Socket
- U20: value MAX232 -> LM386; footprint Package_DIP:DIP-16_W7.62mm_Socket -> Package_DIP:DIP-8_W7.62mm_Socket
- U21: value 74HCT00 -> 74HCT595; footprint Package_DIP:DIP-14_W7.62mm_Socket -> Package_DIP:DIP-16_W7.62mm_Socket
- U22: value SN76489AN -> 74HCT595
- U23: value LM386 -> 74HCT14; footprint Package_DIP:DIP-8_W7.62mm_Socket -> Package_DIP:DIP-14_W7.62mm_Socket
- U3: value 62256 -> W65C22S; footprint Package_DIP:DIP-28_W15.24mm_Socket -> Package_DIP:DIP-40_W15.24mm_Socket
- U4: value 62256 -> 16550; footprint Package_DIP:DIP-28_W15.24mm_Socket -> Package_DIP:DIP-40_W15.24mm_Socket
- U5: value 74HCT00 -> SN76489AN; footprint Package_DIP:DIP-14_W7.62mm_Socket -> Package_DIP:DIP-16_W7.62mm_Socket
- U6: value 2864 -> 62256
- U7: value 74HCT273 -> 62256; footprint Package_DIP:DIP-20_W7.62mm_Socket -> Package_DIP:DIP-28_W15.24mm_Socket
- U8: value 74HCT00 -> 2864; footprint Package_DIP:DIP-14_W7.62mm_Socket -> Package_DIP:DIP-28_W15.24mm_Socket
- U9: value W65C22S -> 62256; footprint Package_DIP:DIP-40_W15.24mm_Socket -> Package_DIP:DIP-28_W15.24mm_Socket
- Y1: value 10.738635Mhz -> 1Mhz; footprint Crystal:Crystal_HC49-4H_Vertical -> Oscillator:Oscillator_DIP-14
- Y2: value 11.0592Mhz -> 4Mhz; footprint Crystal:Crystal_HC49-4H_Vertical -> Oscillator:Oscillator_DIP-8
- Y4: value 1Mhz -> 10.738635Mhz; footprint Oscillator:Oscillator_DIP-14 -> Crystal:Crystal_HC49-4H_Vertical
- moved R14 520.5 mm to (432.1, 424.7)
- moved Y2 509.3 mm to (34.9, 597.7), turned to 0 degrees
- moved C29 500.0 mm to (14.9, 580.3), turned to 0 degrees
- moved Y1 498.3 mm to (434.1, 446.7), turned to 0 degrees
- moved C31 493.1 mm to (14.9, 586.8)
- moved C5 477.1 mm to (33.6, 560.0), turned to 0 degrees
- moved C26 465.8 mm to (414.5, 420.9), turned to 0 degrees
- moved R10 463.1 mm to (69.3, 563.1)
- moved R9 462.5 mm to (69.3, 560.0)
- moved C27 462.3 mm to (414.5, 426.8), turned to 0 degrees
- moved C3 457.0 mm to (396.4, 397.1), turned to 0 degrees
- moved C28 453.9 mm to (51.7, 583.8)
- moved J3 453.1 mm to (391.1, 421.7)
- moved C4 448.2 mm to (396.4, 403.0), turned to 0 degrees
- moved C6 445.6 mm to (396.4, 414.9), turned to 0 degrees
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Connections:
- C20 pad 1: +5V -> Net-(U20-BYPASS)
- C24 pad 1: GND -> +5V
- C24 pad 2: Net-(D1-K) -> GND
- C26 pad 1: Net-(U10-XTAL2) -> GND
- C26 pad 2: GND -> Net-(D1-K)
- C27 pad 1: Net-(U10-XTAL1) -> +5V
- C28 pad 1: Net-(Q1-C) -> +5V
- C29 pad 2: GND -> Net-(C29-Pad2)
- C30 pad 1: Net-(U19-XIN) -> Net-(C30-Pad1)
- C30 pad 2: GND -> Net-(C30-Pad2)
- C31 pad 1: Net-(U20-C1+) -> Net-(C30-Pad1)
- C31 pad 2: Net-(U20-C1-) -> Net-(C31-Pad2)
- C32 pad 1: Net-(U20-C2+) -> Net-(U4-XIN)
- C32 pad 2: Net-(U20-C2-) -> GND
- C33 pad 1: Net-(U20-VS+) -> Net-(C33-Pad1)
- C33 pad 2: +5V -> GND
- C34 pad 1: GND -> Net-(Q1-C)
- C34 pad 2: Net-(U20-VS-) -> GND
- C35 pad 1: Net-(C35-Pad1) -> Net-(U2-XTAL1)
- C35 pad 2: Net-(C35-Pad2) -> GND
- C36 pad 1: Net-(C36-Pad1) -> Net-(U24-C1+)
- C36 pad 2: Net-(C36-Pad2) -> Net-(U24-C1-)
- C37 pad 1: Net-(C35-Pad1) -> Net-(U2-XTAL2)
- C37 pad 2: Net-(C37-Pad2) -> GND
- C38 pad 1: Net-(U23-BYPASS) -> Net-(U24-C2+)
- C38 pad 2: GND -> Net-(U24-C2-)
- J1 pad 1: Net-(J1-CD/DAT3) -> Net-(J1-Pad1)
- J1 pad 2: Net-(J1-CMD) -> unconnected-(J1-Pad2)
- J1 pad 5: Net-(J1-CLK) -> Net-(J1-Pad5)
- J1 pad 6: GND -> unconnected-(J1-Pad6)
- J2 pad 1: Net-(J2-Pad1) -> +5V
- J2 pad 2: unconnected-(J2-Pad2) -> GND
- J3 pad 1: Net-(J3-In) -> unconnected-(J3-SD-Pad1)
- J3 pad 2: GND -> Net-(J3-CS)
- J4 pad 1: unconnected-(J4-Pad1) -> ~{res}
- J4 pad 2: Net-(U20-T1OUT) -> GND
- J5 pad 1: +5V -> Net-(J5-In)
- LS1 pad 1: Net-(C35-Pad2) -> Net-(C31-Pad2)
- Q1 pad 1: Net-(J3-In) -> Net-(J5-In)
- R1 pad 1: GND -> Net-(J1-Pad1)
- R1 pad 2: Net-(J1-CARD_DETECT) -> +5V
- R10 pad 1: Net-(U19-XOUT) -> GND
- R10 pad 2: Net-(C29-Pad1) -> Net-(C30-Pad2)
- R11 pad 1: Net-(U9-CS1) -> Net-(C33-Pad1)
- R11 pad 2: +5V -> Net-(U4-XIN)
- R12 pad 1: Net-(R12-Pad1) -> Net-(U4-CS0)
- R13 pad 2: Net-(U19-~{DCD}) -> Net-(U4-RD)
- R14 pad 1: Net-(U1-RDY) -> Net-(U4-XOUT)
- R14 pad 2: +5V -> Net-(C33-Pad1)
- R15 pad 1: Net-(U1-BE) -> GND
- R15 pad 2: +5V -> Net-(J5-In)
- R16 pad 1: Net-(U1-~{SO}) -> GND
- R16 pad 2: +5V -> Net-(Q1-B)
- R17 pad 1: Net-(U22-READY) -> GND
- R17 pad 2: +5V -> Net-(U4-~{DCD})
- R2 pad 1: Net-(J2-Pad1) -> Net-(J1-Pad5)
- R3 pad 1: Net-(J2-Pad5) -> Net-(D1-A)
- R3 pad 2: +5V -> Net-(D1-K)
- R4 pad 1: Net-(D1-A) -> Net-(U3-CS1)
- R4 pad 2: Net-(D1-K) -> +5V
- R5 pad 1: GND -> Net-(U1-BE)
- R5 pad 2: Net-(J3-In) -> +5V
- R6 pad 1: GND -> Net-(U1-~{SO})
- R6 pad 2: Net-(Q1-B) -> +5V
- R7 pad 1: Net-(U19-CS0) -> Net-(U1-RDY)
- R8 pad 1: GND -> Net-(R8-Pad1)
- R8 pad 2: Net-(U19-RD) -> +5V
- R9 pad 1: Net-(C29-Pad1) -> Net-(U5-READY)
- R9 pad 2: Net-(U19-XIN) -> +5V
- RV1 pad 1: Net-(U22-AUDIO_OUT) -> Net-(U5-AUDIO_OUT)
- RV1 pad 2: Net-(U23-+) -> Net-(U20-+)
- U10 pad 1: Net-(U10-~{RAS}) -> phi2
- U10 pad 10: /ad0 -> GND
- U10 pad 11: Net-(U10-R/~{W}) -> GND
- U10 pad 12: GND -> ~{rom}
- U10 pad 13: a0 -> ram
- U10 pad 14: Net-(U10-~{CSW}) -> dev0
- U10 pad 15: Net-(U10-~{CSR}) -> ~{dev1}
- U10 pad 16: ~{nmi} -> ~{dev2}
- U10 pad 17: /d7 -> ~{dev3}
- U10 pad 18: /d6 -> ~{dev4}
- U10 pad 19: /d5 -> dev5
- U10 pad 2: Net-(U10-~{CAS}) -> /a15
- U10 pad 20: /d4 -> +5V
- U10 pad 3: /ad7 -> /a14
- U10 pad 4: /ad6 -> /a13
- U10 pad 5: /ad5 -> /a12
- U10 pad 6: /ad4 -> /a11
- U10 pad 7: /ad3 -> /a10
- U10 pad 8: /ad2 -> GND
- U10 pad 9: /ad1 -> GND
- U11 pad 1: /va13 -> ~{res}
- U11 pad 10: /va0 -> GND
- U11 pad 11: /vd0 -> Net-(U11-Cp)
- U11 pad 12: /vd1 -> /bk4
- U11 pad 13: /vd2 -> /d4
- U11 pad 14: GND -> /d5
- U11 pad 15: /vd3 -> /bk5
- U11 pad 16: /vd4 -> /bk6
- U11 pad 17: /vd5 -> /d6
- U11 pad 18: /vd6 -> /d7
- U11 pad 19: /vd7 -> /bk7
- U11 pad 2: /va12 -> /bk0
- U11 pad 20: Net-(U10-~{CAS}) -> +5V
- U11 pad 3: /va7 -> /d0
- U11 pad 4: /va6 -> /d1
- U11 pad 5: /va5 -> /bk1
- U11 pad 6: /va4 -> /bk2
- U11 pad 7: /va3 -> /d2
- U11 pad 8: /va2 -> /d3
- U11 pad 9: /va1 -> /bk3
- U12 pad 1: Net-(U10-~{RAS}) -> ~{res}
- U12 pad 2: Net-(U14-Cp) -> +5V
- U12 pad 3: Net-(U10-~{CAS}) -> GND
- U13 pad 1: Net-(U10-R/~{W}) -> ~{r}/w
- U13 pad 10: GND -> Net-(R8-Pad1)
- U13 pad 11: Net-(U11-~{OE}) -> ~{r}/w
- U13 pad 12: /vd7 -> r/~{w}
- U13 pad 13: /vd6 -> r/~{w}
- U13 pad 14: /vd5 -> +5V
- U13 pad 2: /ad0 -> dev5
- U13 pad 3: /ad1 -> Net-(U11-Cp)
- U13 pad 4: /ad2 -> ~{i0}
- U13 pad 5: /ad3 -> ~{i0}
- U13 pad 6: /ad4 -> Net-(U13-Pad6)
- U13 pad 7: /ad5 -> GND
- U13 pad 8: /ad6 -> Net-(U13-Pad8)
- U13 pad 9: /ad7 -> i1
- U14 pad 1: GND -> /a15
- U14 pad 10: GND -> ram
- U14 pad 11: Net-(U14-Cp) -> ~{irq}
- U14 pad 12: /va6 -> Net-(U13-Pad6)
- U14 pad 13: /va5 -> Net-(U13-Pad8)
- U14 pad 14: /va4 -> +5V
- U14 pad 2: /ad0 -> /a15
- U14 pad 3: /ad1 -> Net-(U14-Pad3)
- U14 pad 4: /ad2 -> Net-(U14-Pad3)
- U14 pad 5: /ad3 -> ram
- U14 pad 6: /ad4 -> Net-(U6-~{CS})
- U14 pad 7: /ad5 -> GND
- U14 pad 8: /ad6 -> Net-(U7-~{CS})
- U14 pad 9: /ad7 -> /a15
- U15 pad 1: GND -> clk
- U15 pad 10: GND -> ~{r}/w
- U15 pad 11: Net-(U15-Cp) -> Net-(U4-~{RD})
- U15 pad 12: /va13 -> r/~{w}
- U15 pad 13: /va12 -> clk
- U15 pad 14: /va11 -> +5V
- U15 pad 2: /ad0 -> r/~{w}
- U15 pad 3: /ad1 -> Net-(U4-~{WR})
- U15 pad 4: /ad2 -> r/~{w}
- U15 pad 5: /ad3 -> dev0
- U15 pad 6: /ad4 -> Net-(U2-~{CSR})
- U15 pad 7: /ad5 -> GND
- U15 pad 8: /ad6 -> Net-(U2-~{CSW})
- U15 pad 9: /ad7 -> dev0
- U16 pad 1: Net-(J2-Pad5) -> Net-(U16-OE)
- U16 pad 10: Net-(U17-SER) -> GND
- U16 pad 11: Net-(U16-Pad11) -> Net-(U16-Cp)
- U16 pad 12: Net-(U16-Pad11) -> /vd7
- U16 pad 13: Net-(J2-Pad1) -> /vd6
- U16 pad 14: +5V -> /vd5
- U16 pad 2: Net-(D1-A) -> /ad0
- U16 pad 3: Net-(D1-K) -> /ad1
- U16 pad 4: Net-(U17-RCLK) -> /ad2
- U16 pad 5: Net-(J2-Pad5) -> /ad3
- U16 pad 6: Net-(U16-Pad6) -> /ad4
- U16 pad 7: GND -> /ad5
- U16 pad 8: Net-(U17-SRCLK) -> /ad6
- U16 pad 9: Net-(U16-Pad6) -> /ad7
- U17 pad 1: unconnected-(U17-QB-Pad1) -> GND
- U17 pad 10: +5V -> GND
- U17 pad 11: Net-(U17-SRCLK) -> Net-(U17-Cp)
- U17 pad 12: Net-(U17-RCLK) -> /va6
- U17 pad 13: GND -> /va5
- U17 pad 14: Net-(U17-SER) -> /va4
- U17 pad 15: unconnected-(U17-QA-Pad15) -> /va3
- U17 pad 16: +5V -> /va2
- U17 pad 2: Net-(U17-QC) -> /ad0
- U17 pad 3: Net-(U17-QD) -> /ad1
- U17 pad 4: Net-(U17-QE) -> /ad2
- U17 pad 5: Net-(U17-QF) -> /ad3
- U17 pad 6: Net-(U17-QG) -> /ad4
- U17 pad 7: Net-(U17-QH) -> /ad5
- U17 pad 8: GND -> /ad6
- U17 pad 9: Net-(U17-QH') -> /ad7
- U18 pad 1: Net-(U18-QB) -> GND
- U18 pad 10: +5V -> GND
- U18 pad 11: Net-(U17-SRCLK) -> Net-(U18-Cp)
- U18 pad 12: Net-(U17-RCLK) -> /va13
- U18 pad 13: GND -> /va12
- U18 pad 14: Net-(U17-QH') -> /va11
- U18 pad 15: Net-(U18-QA) -> /va10
- U18 pad 16: +5V -> /va9
- U18 pad 2: unconnected-(U18-QC-Pad2) -> /ad0
- U18 pad 3: unconnected-(U18-QD-Pad3) -> /ad1
- U18 pad 4: unconnected-(U18-QE-Pad4) -> /ad2
- U18 pad 5: unconnected-(U18-QF-Pad5) -> /ad3
- U18 pad 6: unconnected-(U18-QG-Pad6) -> /ad4
- U18 pad 7: unconnected-(U18-QH-Pad7) -> /ad5
- U18 pad 8: GND -> /ad6
- U18 pad 9: unconnected-(U18-QH'-Pad9) -> /ad7
- U19 pad 1: /d0 -> Net-(U2-~{RAS})
- U19 pad 10: Net-(U19-SIN) -> Net-(U16-Cp)
- U19 pad 11: Net-(U19-SOUT) -> Net-(U16-OE)
- U19 pad 12: Net-(U19-CS0) -> Net-(U4-MR)
- U19 pad 13: Net-(U19-CS0) -> ~{res}
- U19 pad 14: ~{dev2} -> +5V
- U19 pad 2: /d1 -> Net-(U17-Cp)
- U19 pad 3: /d2 -> Net-(U2-~{CAS})
- U19 pad 4: /d3 -> Net-(U19-Pad4)
- U19 pad 5: /d4 -> Net-(U19-Pad4)
- U19 pad 6: /d5 -> Net-(U19-Pad6)
- U19 pad 7: /d6 -> GND
- U19 pad 8: /d7 -> Net-(U18-Cp)
- U19 pad 9: Net-(U19-RCLK) -> Net-(U19-Pad6)
- U2 pad 1: phi2 -> Net-(U2-~{RAS})
- U2 pad 10: GND -> /ad0
- U2 pad 11: GND -> Net-(U16-OE)
- U2 pad 12: ~{rom} -> GND
- U2 pad 13: ram -> a0
- U2 pad 14: dev0 -> Net-(U2-~{CSW})
- U2 pad 15: ~{dev1} -> Net-(U2-~{CSR})
- U2 pad 16: ~{dev2} -> ~{nmi}
- U2 pad 17: ~{dev3} -> /d7
- U2 pad 18: ~{dev4} -> /d6
- U2 pad 19: dev5 -> /d5
- U2 pad 2: /a15 -> Net-(U2-~{CAS})
- U2 pad 20: +5V -> /d4
- U2 pad 3: /a14 -> /ad7
- U2 pad 4: /a13 -> /ad6
- U2 pad 5: /a12 -> /ad5
- U2 pad 6: /a11 -> /ad4
- U2 pad 7: /a10 -> /ad3
- U2 pad 8: GND -> /ad2
- U2 pad 9: GND -> /ad1
- U20 pad 1: Net-(U20-C1+) -> Net-(C29-Pad1)
- U20 pad 2: Net-(U20-VS+) -> GND
- U20 pad 3: Net-(U20-C1-) -> Net-(U20-+)
- U20 pad 4: Net-(U20-C2+) -> GND
- U20 pad 5: Net-(U20-C2-) -> Net-(C30-Pad1)
- U20 pad 6: Net-(U20-VS-) -> +5V
- U20 pad 7: Net-(U20-T2OUT) -> Net-(U20-BYPASS)
- U20 pad 8: Net-(U20-R2IN) -> Net-(C29-Pad2)
- U21 pad 1: clk -> Net-(U21-QB)
- U21 pad 10: Net-(R12-Pad1) -> +5V
- U21 pad 11: ~{irq} -> Net-(U21-SRCLK)
- U21 pad 12: Net-(U21-Pad12) -> Net-(U21-RCLK)
- U21 pad 13: Net-(U21-Pad13) -> GND
- U21 pad 14: +5V -> Net-(U21-SER)
- U21 pad 2: r/~{w} -> unconnected-(U21-QC-Pad2)
- U21 pad 3: Net-(U19-~{WR}) -> unconnected-(U21-QD-Pad3)
- U21 pad 4: ~{i0} -> unconnected-(U21-QE-Pad4)
- U21 pad 5: ~{i0} -> unconnected-(U21-QF-Pad5)
- U21 pad 6: Net-(U21-Pad12) -> unconnected-(U21-QG-Pad6)
- U21 pad 7: GND -> unconnected-(U21-QH-Pad7)
- U21 pad 8: Net-(U21-Pad13) -> GND
- U21 pad 9: i1 -> unconnected-(U21-QH'-Pad9)
- U22 pad 1: /d2 -> unconnected-(U22-QB-Pad1)
- U22 pad 10: /d7 -> +5V
- U22 pad 11: /d6 -> Net-(U21-SRCLK)
- U22 pad 12: /d5 -> Net-(U21-RCLK)
- U22 pad 13: /d4 -> GND
- U22 pad 14: aclk -> Net-(U22-SER)
- U22 pad 15: /d3 -> unconnected-(U22-QA-Pad15)
- U22 pad 2: /d1 -> Net-(U22-QC)
- U22 pad 3: /d0 -> Net-(U22-QD)
- U22 pad 4: Net-(U22-READY) -> Net-(U22-QE)
- U22 pad 5: r/~{w} -> Net-(U22-QF)
- U22 pad 6: ~{dev2} -> Net-(U22-QG)
- U22 pad 7: Net-(U22-AUDIO_OUT) -> Net-(U22-QH)
- U22 pad 9: unconnected-(U22-NC-Pad9) -> Net-(U21-SER)
- U23 pad 1: Net-(C36-Pad1) -> Net-(J1-Pad5)
- U23 pad 2: GND -> Net-(D1-A)
- U23 pad 3: Net-(U23-+) -> Net-(D1-K)
- U23 pad 4: GND -> Net-(U21-RCLK)
- U23 pad 5: Net-(C35-Pad1) -> Net-(J1-Pad5)
- U23 pad 6: +5V -> Net-(U23-Pad6)
- U23 pad 7: Net-(U23-BYPASS) -> GND
- U23 pad 8: Net-(C36-Pad2) -> Net-(U21-SRCLK)
- U3 pad 1: /a14 -> GND
- U3 pad 10: a0 -> Net-(U21-QB)
- U3 pad 11: /d0 -> Net-(U21-QA)
- U3 pad 12: /d1 -> Net-(U22-QH)
- U3 pad 13: /d2 -> Net-(U22-QG)
- U3 pad 14: GND -> Net-(U22-QF)
- U3 pad 15: /d3 -> Net-(U22-QE)
- U3 pad 16: /d4 -> Net-(U22-QD)
- U3 pad 17: /d5 -> Net-(U22-QC)
- U3 pad 18: /d6 -> Net-(U21-RCLK)
- U3 pad 19: /d7 -> unconnected-(U3-CB2-Pad19)
- U3 pad 2: /a12 -> Net-(J3-CS)
- U3 pad 20: Net-(U3-~{CS}) -> +5V
- U3 pad 21: /a10 -> ~{i0}
- U3 pad 22: Net-(U3-~{CS}) -> r/~{w}
- U3 pad 23: /a11 -> ~{dev1}
- U3 pad 24: /a9 -> Net-(U3-CS1)
- U3 pad 25: /a8 -> phi2
- U3 pad 26: /a13 -> /d7
- U3 pad 27: r/~{w} -> /d6
- U3 pad 28: +5V -> /d5
- U3 pad 3: /a7 -> Net-(J3-CLK)
- U3 pad 4: /a6 -> Net-(J3-DI)
- U3 pad 5: /a5 -> unconnected-(U3-PA3-Pad5)
- U3 pad 6: /a4 -> unconnected-(U3-PA4-Pad6)
- U3 pad 7: /a3 -> unconnected-(U3-PA5-Pad7)
- U3 pad 8: /a2 -> unconnected-(U3-PA6-Pad8)
- U3 pad 9: /a1 -> Net-(J3-DO)
- U4 pad 1: /bk1 -> /d0
- U4 pad 10: a0 -> Net-(U24-R1OUT)
- U4 pad 11: /d0 -> Net-(U24-T1IN)
- U4 pad 12: /d1 -> Net-(U4-CS0)
- U4 pad 13: /d2 -> Net-(U4-CS0)
- U4 pad 14: GND -> ~{dev1}
- U4 pad 15: /d3 -> Net-(U4-RCLK)
- U4 pad 16: /d4 -> Net-(U4-XIN)
- U4 pad 17: /d5 -> Net-(U4-XOUT)
- U4 pad 18: /d6 -> Net-(U4-~{WR})
- U4 pad 19: /d7 -> Net-(U4-RD)
- U4 pad 2: /a12 -> /d1
- U4 pad 20: Net-(U4-~{CS}) -> GND
- U4 pad 21: /a10 -> Net-(U4-~{RD})
- U4 pad 22: Net-(U4-~{CS}) -> Net-(U4-RD)
- U4 pad 23: /a11 -> unconnected-(U4-DDIS-Pad23)
- U4 pad 24: /a9 -> unconnected-(U4-~{TXRDY}-Pad24)
- U4 pad 25: /a8 -> Net-(U4-RD)
- U4 pad 26: /bk0 -> /a2
- U4 pad 27: r/~{w} -> /a1
- U4 pad 28: +5V -> a0
- U4 pad 3: /a7 -> /d2
- U4 pad 4: /a6 -> /d3
- U4 pad 5: /a5 -> /d4
- U4 pad 6: /a4 -> /d5
- U4 pad 7: /a3 -> /d6
- U4 pad 8: /a2 -> /d7
- U4 pad 9: /a1 -> Net-(U4-RCLK)
- U5 pad 1: /a15 -> /d2
- U5 pad 10: ram -> /d7
- U5 pad 11: ~{r}/w -> /d6
- U5 pad 12: r/~{w} -> /d5
- U5 pad 13: r/~{w} -> /d4
- U5 pad 14: +5V -> Net-(U5-CLOCK)
- U5 pad 2: /a15 -> /d1
- U5 pad 3: Net-(U5-Pad3) -> /d0
- U5 pad 4: Net-(U5-Pad3) -> Net-(U5-READY)
- U5 pad 5: ram -> r/~{w}
- U5 pad 6: Net-(U3-~{CS}) -> ~{dev2}
- U5 pad 7: GND -> Net-(U5-AUDIO_OUT)
- U5 pad 8: Net-(U4-~{CS}) -> GND
- U5 pad 9: /a15 -> unconnected-(U5-NC-Pad9)
- U6 pad 1: unconnected-(U6-NC-Pad1) -> /a14
- U6 pad 20: ~{rom} -> Net-(U6-~{CS})
- U6 pad 22: ~{rom} -> Net-(U6-~{CS})
- U6 pad 26: unconnected-(U6-NC-Pad26) -> /a13
- U6 pad 27: +5V -> r/~{w}
- U7 pad 1: ~{res} -> /bk1
- U7 pad 10: GND -> a0
- U7 pad 11: Net-(U7-Cp) -> /d0
- U7 pad 12: /bk4 -> /d1
- U7 pad 13: /d4 -> /d2
- U7 pad 14: /d5 -> GND
- U7 pad 15: /bk5 -> /d3
- U7 pad 16: /bk6 -> /d4
- U7 pad 17: /d6 -> /d5
- U7 pad 18: /d7 -> /d6
- U7 pad 19: /bk7 -> /d7
- U7 pad 2: /bk0 -> /a12
- U7 pad 20: +5V -> Net-(U7-~{CS})
- U7 pad 3: /d0 -> /a7
- U7 pad 4: /d1 -> /a6
- U7 pad 5: /bk1 -> /a5
- U7 pad 6: /bk2 -> /a4
- U7 pad 7: /d2 -> /a3
- U7 pad 8: /d3 -> /a2
- U7 pad 9: /bk3 -> /a1
- U8 pad 1: ~{r}/w -> unconnected-(U8-NC-Pad1)
- U8 pad 10: ~{r}/w -> a0
- U8 pad 11: Net-(U19-~{RD}) -> /d0
- U8 pad 12: r/~{w} -> /d1
- U8 pad 13: clk -> /d2
- U8 pad 14: +5V -> GND
- U8 pad 2: dev5 -> /a12
- U8 pad 3: Net-(U7-Cp) -> /a7
- U8 pad 4: r/~{w} -> /a6
- U8 pad 5: dev0 -> /a5
- U8 pad 6: Net-(U10-~{CSR}) -> /a4
- U8 pad 7: GND -> /a3
- U8 pad 8: Net-(U10-~{CSW}) -> /a2
- U8 pad 9: dev0 -> /a1
- U9 pad 1: GND -> /va13
- U9 pad 10: Net-(U18-QB) -> /va0
- U9 pad 11: Net-(U18-QA) -> /vd0
- U9 pad 12: Net-(U17-QH) -> /vd1
- U9 pad 13: Net-(U17-QG) -> /vd2
- U9 pad 14: Net-(U17-QF) -> GND
- U9 pad 15: Net-(U17-QE) -> /vd3
- U9 pad 16: Net-(U17-QD) -> /vd4
- U9 pad 17: Net-(U17-QC) -> /vd5
- U9 pad 18: Net-(U17-RCLK) -> /vd6
- U9 pad 19: unconnected-(U9-CB2-Pad19) -> /vd7
- U9 pad 2: Net-(J1-CD/DAT3) -> /va12
- U9 pad 20: +5V -> Net-(U2-~{CAS})
- U9 pad 21: ~{i0} -> /va10
- U9 pad 22: r/~{w} -> Net-(U16-Cp)
- U9 pad 23: ~{dev1} -> /va11
- U9 pad 24: Net-(U9-CS1) -> /va9
- U9 pad 25: phi2 -> /va8
- U9 pad 26: /d7 -> /va13
- U9 pad 27: /d6 -> Net-(U16-OE)
- U9 pad 28: /d5 -> +5V
- U9 pad 3: Net-(J1-CLK) -> /va7
- U9 pad 4: Net-(J1-CMD) -> /va6
- U9 pad 5: unconnected-(U9-PA3-Pad5) -> /va5
- U9 pad 6: unconnected-(U9-PA4-Pad6) -> /va4
- U9 pad 7: unconnected-(U9-PA5-Pad7) -> /va3
- U9 pad 8: unconnected-(U9-PA6-Pad8) -> /va2
- U9 pad 9: Net-(J1-CMD) -> /va1
- Y1 pad 1: Net-(U10-XTAL1) -> unconnected-(Y1-NC-Pad1)
- Y2 pad 1: Net-(U19-XIN) -> unconnected-(Y2-EN-Pad1)
- Y4 pad 1: unconnected-(Y4-NC-Pad1) -> Net-(U2-XTAL1)
Routing:
- net +5V: track 939.4 -> 69.6 mm, vias 2 -> 0
- net GND: track 753.9 -> 0.00 mm, vias 69 -> 0
- net /d7: track 461.3 -> 0.00 mm, vias 6 -> 0
- net /d5: track 459.4 -> 0.00 mm, vias 5 -> 0
- net /d6: track 457.2 -> 0.00 mm, vias 4 -> 0
- net /d4: track 426.7 -> 0.00 mm, vias 3 -> 0
- net /d0: track 411.6 -> 0.00 mm, vias 5 -> 0
- net /d1: track 410.3 -> 0.00 mm, vias 3 -> 0
- net /d3: track 399.6 -> 0.00 mm, vias 2 -> 0
- net a0: track 398.6 -> 0.00 mm, vias 2 -> 0
- net /d2: track 386.0 -> 0.00 mm, vias 3 -> 0
- net ~{res}: track 321.6 -> 0.00 mm, vias 2 -> 0
- net r/~{w}: track 319.4 -> 0.00 mm
- net /a2: track 308.8 -> 0.00 mm, vias 1 -> 0
- net /a1: track 308.0 -> 0.00 mm, vias 5 -> 0
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Other:
- board size 195.6 x 149.9 mm -> 304.8 x 203.2 mm

Commit message: hw: update PCB
Parts:
- moved C21 563.2 mm to (-77.2, 671.7)
- moved C22 563.2 mm to (-77.2, 677.6)
- moved C23 563.2 mm to (-77.2, 683.6)
- moved C25 563.2 mm to (-114.1, 697.3)
- moved C26 563.2 mm to (-77.2, 695.5)
- moved C3 563.2 mm to (-95.3, 671.7)
- moved D1 563.2 mm to (-49.0, 679.6)
- moved J1 563.2 mm to (-48.3, 659.1)
- moved J3 563.2 mm to (-100.6, 696.3)
- moved R1 563.2 mm to (-59.7, 658.4)
- moved R2 563.2 mm to (-59.7, 661.5)
- moved R3 563.2 mm to (-59.7, 664.7)
- moved R4 563.2 mm to (-59.7, 667.8)
- moved U21 563.2 mm to (-83.6, 625.9)
- moved U22 563.2 mm to (-71.9, 625.9)
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Routing:
- net /a11: track 0.00 -> 189.6 mm
- net /a10: track 0.00 -> 189.4 mm
- net +5V: track 69.6 -> 220.4 mm
- net /a9: track 0.00 -> 137.1 mm
- net a0: track 0.00 -> 132.3 mm
- net /d3: track 0.00 -> 127.5 mm, vias 0 -> 1
- net /d2: track 0.00 -> 127.1 mm, vias 0 -> 1
- net /d1: track 0.00 -> 127.1 mm, vias 0 -> 1
- net /d0: track 0.00 -> 127.1 mm, vias 0 -> 1
- net /a1: track 0.00 -> 126.8 mm
- net /a8: track 0.00 -> 125.0 mm
- net /d4: track 0.00 -> 122.8 mm, vias 0 -> 1
- net /a2: track 0.00 -> 120.9 mm
- net /d5: track 0.00 -> 117.3 mm, vias 0 -> 1
- net /a3: track 0.00 -> 115.4 mm
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
Commit message: vm/hw: simplify hw. remove bank switch flip-flop in favor of VIA pin
Parts:
- removed C11, C14, C28: 0.1uF, Capacitor_THT:C_Disc_D7.5mm_W4.4mm_P5.00mm
- removed R8: 10K, Resistor_THT:R_Axial_DIN0204_L3.6mm_D1.6mm_P7.62mm_Horizontal
- removed U11: 74HCT273, Package_DIP:DIP-20_W7.62mm_Socket
- removed U14: 74HCT00, Package_DIP:DIP-14_W7.62mm_Socket
- removed Y2: 4Mhz, Oscillator:Oscillator_DIP-8
- added R18: 10K, Resistor_THT:R_Axial_DIN0204_L3.6mm_D1.6mm_P7.62mm_Horizontal, F.Cu at (-175.9, 533.2)
- moved C29 534.9 mm to (247.8, 488.1)
- moved C31 534.9 mm to (247.8, 494.6)
- moved LS1 533.8 mm to (247.5, 540.3)
- moved C5 495.4 mm to (220.6, 493.1)
- moved U20 490.0 mm to (221.8, 540.1)
- moved C30 489.7 mm to (238.7, 481.2)
- moved C20 488.1 mm to (229.6, 481.2)
- moved RV1 477.1 mm to (233.7, 540.3)
- moved R10 450.0 mm to (209.5, 495.6)
- moved R9 450.0 mm to (209.5, 492.4)
- moved U13 447.9 mm to (2.18, 544.3)
- moved U5 438.6 mm to (214.6, 518.2), turned to 0 degrees
- moved U12 402.8 mm to (82.0, 559.9)
- moved J4 372.9 mm to (73.8, 551.8)
- moved J2 372.9 mm to (69.2, 551.8)
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Connections:
- U10 pad 13: ram -> ~{ramlo}
- U10 pad 14: dev0 -> ~{ramhi}
- U10 pad 15: ~{dev1} -> dev0
- U10 pad 16: ~{dev2} -> ~{dev1}
- U10 pad 17: ~{dev3} -> ~{dev2}
- U10 pad 18: ~{dev4} -> ~{dev3}
- U10 pad 19: dev5 -> ~{dev4}
- U13 pad 1: ~{r}/w -> ~{i0}
- U13 pad 10: Net-(R8-Pad1) -> Net-(U13-Pad10)
- U13 pad 11: ~{r}/w -> Net-(U2-~{CSW})
- U13 pad 12: r/~{w} -> dev0
- U13 pad 13: r/~{w} -> Net-(U13-Pad13)
- U13 pad 2: dev5 -> ~{i0}
- U13 pad 3: Net-(U11-Cp) -> Net-(U13-Pad3)
- U13 pad 4: ~{i0} -> i1
- U13 pad 5: ~{i0} -> +5V
- U13 pad 6: Net-(U13-Pad6) -> Net-(U13-Pad10)
- U13 pad 8: Net-(U13-Pad8) -> ~{irq}
- U13 pad 9: i1 -> Net-(U13-Pad3)
- U15 pad 1: clk -> r/~{w}
- U15 pad 10: ~{r}/w -> ~{res}
- U15 pad 11: Net-(U4-~{RD}) -> Net-(U2-~{CSR})
- U15 pad 13: clk -> dev0
- U15 pad 2: r/~{w} -> clk
- U15 pad 3: Net-(U4-~{WR}) -> Net-(U4-~{RD})
- U15 pad 4: r/~{w} -> clk
- U15 pad 5: dev0 -> r/~{w}
- U15 pad 6: Net-(U2-~{CSR}) -> Net-(U4-~{WR})
- U15 pad 8: Net-(U2-~{CSW}) -> Net-(U4-MR)
- U15 pad 9: dev0 -> ~{res}
- U19 pad 12: Net-(U4-MR) -> Net-(U13-Pad13)
- U19 pad 13: ~{res} -> r/~{w}
- U2 pad 38: unconnected-(U2-CPUCLK-Pad38) -> aclk
- U3 pad 39: unconnected-(U3-CA2-Pad39) -> bk
- U5 pad 14: Net-(U5-CLOCK) -> aclk
- U6 pad 20: Net-(U6-~{CS}) -> ~{ramlo}
- U6 pad 22: Net-(U6-~{CS}) -> ~{ramlo}
- U7 pad 1: /bk1 -> bk
- U7 pad 20: Net-(U7-~{CS}) -> ~{ramhi}
- U7 pad 22: Net-(U7-~{CS}) -> ~{ramhi}
- U7 pad 26: /bk0 -> /a13
Routing:
- net ~{ramlo}: track 0.00 -> 70.0 mm, vias 0 -> 2
- net ~{rom}: track 0.00 -> 63.4 mm, vias 0 -> 2
- net ~{ramhi}: track 0.00 -> 55.5 mm, vias 0 -> 2
- net /d2: track 127.1 -> 167.5 mm
- net /d0: track 127.1 -> 167.5 mm
- net /d1: track 127.1 -> 167.5 mm
- net /d3: track 127.5 -> 151.1 mm
- net a0: track 132.3 -> 151.9 mm
- net /a3: track 115.4 -> 135.0 mm
- net /a2: track 120.9 -> 140.5 mm
- net /a1: track 126.8 -> 146.4 mm
- net /a13: track 47.4 -> 66.5 mm
- net /a14: track 60.0 -> 78.0 mm, vias 1 -> 0
- net /d7: track 106.3 -> 115.2 mm
- net /d4: track 122.8 -> 131.7 mm
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
Commit message: hw: update pcb
Parts:
- J2: value POWER -> +5V
- moved J2 533.5 mm to (107.3, 19.7), turned to 90 degrees
- moved J4 532.6 mm to (97.2, 19.7), turned to 90 degrees
- moved U12 525.7 mm to (91.4, 34.3), turned to -90 degrees
- moved R18 491.1 mm to (104.8, 130.2), turned to 90 degrees
- moved U3 483.3 mm to (85.7, 120.0)
- moved U15 482.8 mm to (134.6, 76.8)
- moved U13 481.6 mm to (118.1, 76.8)
- moved C12 477.2 mm to (97.2, 35.6), turned to 90 degrees
- moved J3 476.4 mm to (55.2, 120.0)
- moved U21 474.0 mm to (71.1, 122.6)
- moved U23 468.3 mm to (55.2, 153.0)
- moved C15 459.7 mm to (142.2, 71.8), turned to 180 degrees
- moved D1 458.9 mm to (49.5, 158.1), turned to 180 degrees
- moved J1 458.6 mm to (27.3, 148.0)
- moved C21 453.7 mm to (78.7, 117.5), turned to 180 degrees
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Connections:
- U4 pad 14: ~{dev1} -> ~{dev3}
Routing:
- net +5V: track 221.2 -> 1024.3 mm
- net /d7: track 115.2 -> 210.8 mm, vias 1 -> 2
- net /d6: track 120.7 -> 209.5 mm, vias 1 -> 2
- net /d5: track 126.2 -> 209.5 mm, vias 1 -> 2
- net /d4: track 131.7 -> 209.5 mm, vias 1 -> 2
- net /d3: track 151.1 -> 213.0 mm, vias 1 -> 2
- net ~{res}: track 0.00 -> 57.1 mm
- net aclk: track 0.00 -> 54.0 mm, vias 0 -> 1
- net Net-(J1-Pad5): track 0.00 -> 49.7 mm
- net Net-(J1-Pad1): track 0.00 -> 42.4 mm
- net /d0: track 167.5 -> 209.1 mm, vias 1 -> 2
- net /d1: track 167.5 -> 203.6 mm, vias 1 -> 2
- net Net-(U20-+): track 0.00 -> 30.5 mm
- net /d2: track 167.5 -> 197.0 mm, vias 1 -> 2
- net Net-(D1-K): track 0.00 -> 23.6 mm
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Other:
- board size 304.8 x 203.2 mm -> 203.2 x 165.1 mm

Commit message: hw: complete layout
Parts:
- added C11: 0.1uF, Capacitor_THT:C_Disc_D7.5mm_W4.4mm_P5.00mm, F.Cu at (125.7, 41.9)
- added R19: 91K, Resistor_THT:R_Axial_DIN0204_L3.6mm_D1.6mm_P7.62mm_Horizontal, F.Cu at (117.5, 39.4)
- added R20: 27K, Resistor_THT:R_Axial_DIN0204_L3.6mm_D1.6mm_P7.62mm_Horizontal, F.Cu at (117.5, 41.9)
- added R8: 10K, Resistor_THT:R_Axial_DIN0204_L3.6mm_D1.6mm_P7.62mm_Horizontal, F.Cu at (140.3, 95.9)
- J2: value +5V -> LM73100 Breakout; footprint Connector_PinHeader_2.54mm:PinHeader_1x02_P2.54mm_Vertical -> Connector_PinHeader_2.54mm:PinHeader_1x09_P2.54mm_Vertical
- U12: value ~ -> DS1813
- moved R17 51.3 mm to (152.4, 116.2), turned to -90 degrees
- moved R18 18.9 mm to (91.4, 116.8), turned to 0 degrees
- moved C39 18.5 mm to (170.8, 153.0), turned to 90 degrees
- moved U15 18.4 mm to (116.2, 76.8)
- moved C15 18.4 mm to (123.8, 71.8), turned to 90 degrees
- moved C19 16.9 mm to (148.6, 22.2)
- moved U19 16.9 mm to (141.0, 27.3)
- moved J2 15.5 mm to (109.9, 34.9)
- moved C13 14.6 mm to (140.3, 71.7), turned to 90 degrees
- moved U13 14.6 mm to (132.7, 76.8)
- moved U12 9.34 mm to (95.2, 25.8), turned to 0 degrees
- moved C38 9.02 mm to (151.8, 158.1)
- moved C6 6.99 mm to (33.0, 71.8)
- moved C40 5.17 mm to (151.8, 165.7)
- moved R12 5.12 mm to (121.9, 149.9)
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Connections:
- J2 pad 1: +5V -> Net-(J2-Vin)
- U13 pad 10: Net-(U13-Pad10) -> ~{i2}
- U13 pad 4: i1 -> Net-(U13-Pad3)
- U13 pad 5: +5V -> i1
- U13 pad 6: Net-(U13-Pad10) -> Net-(U13-Pad6)
- U13 pad 9: Net-(U13-Pad3) -> Net-(U13-Pad6)
Routing:
- net r/~{w}: track 81.8 -> 473.6 mm, vias 1 -> 4
- net +5V: track 1024.3 -> 1369.4 mm
- net ~{res}: track 57.1 -> 344.4 mm, vias 0 -> 4
- net a0: track 138.2 -> 343.4 mm, vias 0 -> 3
- net ~{dev2}: track 0.01 -> 186.6 mm, vias 0 -> 2
- net ~{nmi}: track 0.00 -> 176.0 mm, vias 0 -> 2
- net phi2: track 28.2 -> 203.0 mm, vias 1 -> 3
- net ~{dev1}: track 0.00 -> 165.7 mm, vias 0 -> 2
- net ~{irq}: track 0.00 -> 161.5 mm, vias 0 -> 2
- net ~{dev3}: track 0.00 -> 161.0 mm, vias 0 -> 3
- net Net-(U2-~{CAS}): track 0.00 -> 157.6 mm, vias 0 -> 1
- net /a1: track 134.2 -> 284.0 mm, vias 0 -> 2
- net /a2: track 127.6 -> 277.2 mm, vias 0 -> 2
- net ~{i0}: track 0.00 -> 137.0 mm, vias 0 -> 2
- net Net-(U4-~{RD}): track 0.00 -> 115.2 mm, vias 0 -> 2
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
Commit message: hw: final?
Parts:
- moved LS1 0.63 mm to (201.9, 139.1)
Routing:
- net ~{dev2}: track 186.6 -> 193.0 mm
- net Net-(U4-~{RD}): track 115.2 -> 110.5 mm
- net clk: track 114.0 -> 118.7 mm
- net ~{dev3}: track 161.0 -> 164.3 mm
- net ~{res}: track 344.4 -> 341.7 mm
- net Net-(U13-Pad13): track 61.9 -> 59.3 mm, vias 1 -> 0
- net r/~{w}: track 473.6 -> 472.2 mm
- net ~{nmi}: track 176.0 -> 174.8 mm
- net Net-(U2-~{RAS}): track 50.6 -> 49.5 mm
- net Net-(U2-~{CAS}): track 157.6 -> 156.5 mm
- net Net-(J5-In): track 19.4 -> 18.5 mm
- net ~{irq}: track 161.5 -> 162.4 mm
- net ~{dev1}: track 165.7 -> 166.6 mm
- net phi2: track 203.0 -> 202.1 mm
- net Net-(Q1-B): track 26.7 -> 26.0 mm
- added copper zone on F.Cu, net GND
Other:
- board text added: "(float) / \"
- board text added: "+5V"
- board text added: "+5Vin"
- board text added: "+5Vout"
- board text added: ".1uF"
- board text added: "10.738635Mhz"
- board text added: "10K"
- board text added: "10R"
- board text added: "10uF"
- board text added: "11.0592Mhz"
- board text added: "16C550A"
- board text added: "1M"
- board text added: "1Mhz"
- board text added: "1N4148 -^"
- board text added: "220uF"
- board text added: "27K"
- board text added: "27pF"
- board text added: "2864"
- board text added: "2N4401-^"
- board text added: "30pF"
- board text added: "5.6K"
- board text added: "62256"
- board text added: "74HCT00"
- board text added: "74HCT04"
- board text added: "74HCT14"
- board text added: "74HCT574"
- board text added: "74HCT595"
- board text added: "75K"
- board text added: "91K"
- board text added: ":-)"
- board text added: "ATF16V8"
- board text added: "CLK"
- board text added: "CS"
- board text added: "DS1813-^"
- board text added: "DVDT"
- board text added: "GND"
- board text added: "IMON (>gnd)"
- board text added: "KBD (PS/2)"
- board text added: "LM386"
- board text added: "LM73100 Breakout"
- board text added: "MAX232"
- board text added: "MISO"
- board text added: "MOSI"
- board text added: "OVLO"
- board text added: "PG"
- board text added: "PGTH"
- board text added: "RESET"
- board text added: "RS232"
- board text added: "SD (SPI) Breakout"
- board text added: "SN76489AN"
- board text added: "SPK"
- board text added: "TMS9918A"
- board text added: "TV (Composite)"
- board text added: "UVLO (tiehi)"
- board text added: "Vol (10K)"
- board text added: "W65C02S"
- board text added: "W65C22S"
